File: kimchi_ulid.kicad_sch (KiCad schematic)
At the start: 59 parts, among them J1 DF40HC(3.5)-60DS, J2 DF40HC(3.5)-60DS, J3 HDMI_A_1.4, J5 Flash, K1 KIMCHI_MICRO, Q1 2N7002, Q2 2N7002, U1 24C32, U2 LM3880, U3 LD3985M27R_SOT23, U4 LD3985M27R_SOT23, U5 LIFCL40-NX, U6 W25Q32JVSS, U7 74AUC1G17

Commit message: Update routing
Parts:
- removed U7: 74AUC1G17, Package_TO_SOT_SMD:SOT-23-5, symbol 74xGxx:74AUC1G17
- added C23: C, Capacitor_SMD:C_0402_1005Metric, symbol Device:C
- added C24, C25, C26: 4.7uF, Capacitor_SMD:C_0603_1608Metric, symbol Device:C
- added C27, C28, C29: 0.01uF, Capacitor_SMD:C_0402_1005Metric, symbol Device:C
- added C30, C34, C35: 0.1uF, Capacitor_SMD:C_0402_1005Metric, symbol Device:C
- added C31, C32, C33: 10uF, Capacitor_SMD:C_0603_1608Metric, symbol Device:C
- added J?: Jtag, Connector_PinHeader_2.54mm:PinHeader_1x07_P2.54mm_Vertical, symbol Connector_Generic:Conn_01x07
- added R15: 100R, Resistor_SMD:R_0402_1005Metric, symbol Device:R
- added R16: R, Resistor_SMD:R_0402_1005Metric, symbol Device:R
- added R17, R18, R22: R, symbol Device:R
- added U10, U9: TPD4E02B04DQA, Package_SON:USON-10_2.5x1.0mm_P0.5mm, symbol Power_Protection:TPD4E02B04DQA
- added U11: LD3985M27R_SOT23, Package_TO_SOT_SMD:SOT-23-5, symbol Regulator_Linear:LD3985M27R_SOT23
- added U7: 74LVC2G17, symbol 74xGxx:74LVC2G17
- added U8: 74LVC1G125, Package_TO_SOT_SMD:SOT-23-5, symbol 74xGxx:74LVC1G125
- J5: footprint Pin_Headers:Pin_Header_Straight_1x07 -> Connector_PinHeader_2.54mm:PinHeader_1x07_P2.54mm_Vertical
Connections:
- net +1V0: now also C31.1
- net +1V8: now also C33.1, C34.1, C35.1, U7.5 (VCC), U7.5 (VCC)
- net +3V3: now also C30.1, C32.1, U11.5 (VOUT)
- net GND: now also U2.2 (GND), C23.2, C24.2, C25.2, C26.2, C27.2, C28.2, C29.2, C30.2, C31.2, C32.2, C33.2, C34.2, C35.2, J?.7 (Pin_7), U10.3 (G), U10.8 (G), U11.2 (GND), U7.2 (GND), U7.2 (GND), U8.3 (GND), U9.3 (G), U9.8 (G)
- net VDD_3V3: now also U2.1 (VCC), C24.1, C25.1, R16.1, R17.1, R18.1, R22.1
- net VDD_5V: now also C26.1, U11.1 (VIN)
- net _tmds_clk+: now also U10.4 (IO3)
- net _tmds_clk-: now also U10.5 (IO4)
- net _tmds_d0+: now also U10.1 (IO1)
- net _tmds_d0-: now also U10.2 (IO2)
- net _tmds_d1+: now also U9.4 (IO3)
- net _tmds_d1-: now also U9.5 (IO4)
- net _tmds_d2+: now also U9.1 (IO1)
- net _tmds_d2-: now also U9.2 (IO2)
- net VDD: now reaches J3.18 (+5V), R12.2, R13.2
- net VDD: now also U8.5 (VDD)
- net en0: now reaches U3.3 (INH)
- net en0: now also U2.6 (FLAG1), R17.2
- net at U3.4 (BYP): now also C27.1
- net at J3.13 (CEC): now also R15.1
- net at J3.19 (HPD/HEAC-), R14.2: now also U7.3
- net en1: now reaches U4.3 (INH)
- net en1: now also U2.5 (FLAG2), R18.2
- net at U4.4 (BYP): now also C28.1
- net at U5.19 (PB10A/PCLKT5_2/ADC_CP2/COMP3P): now also U7.4
- net at U5.24 (PB58A/PCLKT3_1/ADC_CP6): now also U8.1
- net at U5.25 (PB58B/PCLKC3_1/ADC_CN6): now also U8.2
- net at U5.27 (PB68A/ADC_CP8): now also U7.6
- net at U2.3 (EN): now also C23.1, R16.2
- net en2: now reaches U2.4 (FLAG3)
- net en2: now also R22.2, U11.3 (INH)
- new net: R15.2, U7.1, U8.4
- new net: C29.1, U11.4 (BYP)
Other:
- moved on the sheet: Q1, Q2, R1, R10, R11, R12, R13, R14, R2, R3, R4, R5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

Commit message: Update
- Complete inital routing
- Render a board view and update readme
Parts:
- gave numbers to parts that had none: 1
Connections:
- net +3V3: now also J4.7 (Pin_7), R19.1
- net GND: now also J4.6 (Pin_6); no longer J4.7 (Pin_7), R19.1
- net IO: now reaches J4.1 (Pin_1)
- net IO: now also U5.42 (PR11A/SDA/USER_SDA)
- net TMS: now reaches J4.2 (Pin_2)
- net TMS: now also U5.48 (PR6B/TMS/SCSN)
- net TDI: now reaches J4.3 (Pin_3)
- net TDI: now also U5.46 (PR8B/TDI/SSI)
- net TDO: now reaches J4.4 (Pin_4)
- net TDO: now also U5.45 (PR10B/TDO/SSO)
- net TCK: now reaches J4.5 (Pin_5)
- net TCK: now also U5.41 (PR13A/TCK/SCLK/PMU_EXT_CLK)
Changed lines of the file:
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@@
     (stroke (width 0) (type solid) (color 0 0 0 0))
   )
+  (wire (pts (xy 27.94 205.74) (xy 27.94 207.01))
+    (stroke (width 0) (type solid) (color 0 0 0 0))
+  )
   (wire (pts (xy 27.94 247.65) (xy 27.94 246.38))
     (stroke (width 0) (type solid) (color 0 0 0 0))
@@
     (stroke (width 0) (type solid) (color 0 0 0 0))
   )
+  (wire (pts (xy 284.48 226.06) (xy 290.83 226.06))
+    (stroke (width 0) (type solid) (color 0 0 0 0))
+  )
   (wire (pts (xy 285.75 39.37) (xy 274.32 39.37))
     (stroke (width 0) (type solid) (color 0 0 0 0))
@@
     (stroke (width 0) (type solid) (color 0 0 0 0))
   )
-  (wire (pts (xy 288.29 223.52) (xy 290.83 223.52))
+  (wire (pts (xy 288.29 223.52) (xy 288.29 228.6))
     (stroke (width 0) (type solid) (color 0 0 0 0))
   )
-  (wire (pts (xy 288.29 226.06) (xy 288.29 228.6))
+  (wire (pts (xy 288.29 223.52) (xy 290.83 223.52))
     (stroke (width 0) (type solid) (color 0 0 0 0))
   )
@@
     (stroke (width 0) (type solid) (color 0 0 0 0))
   )
-  (wire (pts (xy 290.83 226.06) (xy 288.29 226.06))
-    (stroke (width 0) (type solid) (color 0 0 0 0))
-  )
   (wire (pts (xy 290.83 240.03) (xy 288.29 240.03))
     (stroke (width 0) (type solid) (color 0 0 0 0))
@@
     (effects (font (size 1.27 1.27)) (justify right bottom))
   )
+  (label "TCK" (at 43.18 209.55 180)
+    (effects (font (size 1.27 1.27)) (justify right bottom))
+  )
+  (label "IO" (at 43.18 212.09 180)
+    (effects (font (size 1.27 1.27)) (justify right bottom))
+  )
+  (label "TDO" (at 43.18 217.17 180)
+    (effects (font (size 1.27 1.27)) (justify right bottom))
+  )
+  (label "TDI" (at 43.18 219.71 180)
+    (effects (font (size 1.27 1.27)) (justify right bottom))
+  )
+  (label "TMS" (at 43.18 222.25 180)
+    (effects (font (size 1.27 1.27)) (justify right bottom))
+  )
   (label "FLASH_MISO|IO1" (at 45.72 224.79 180)
     (effects (font (size 1.27 1.27)) (justify right bottom))
@@
     (effects (font (size 1.27 1.27)) (justify right bottom))
   )
+  (label "IO" (at 288.29 210.82 180)
+    (effects (font (size 1.27 1.27)) (justify right bottom))
+  )
+  (label "TMS" (at 288.29 213.36 180)
+    (effects (font (size 1.27 1.27)) (justify right bottom))
+  )
+  (label "TDI" (at 288.29 215.9 180)
+    (effects (font (size 1.27 1.27)) (justify right bottom))
+  )
+  (label "TDO" (at 288.29 218.44 180)
+    (effects (font (size 1.27 1.27)) (justify right bottom))
+  )
+  (label "TCK" (at 288.29 220.98 180)
+    (effects (font (size 1.27 1.27)) (justify right bottom))
+  )
   (label "FLASH_CS" (at 288.29 240.03 180)
     (effects (font (size 1.27 1.27)) (justify right bottom))
@@
     (pin "1")
   )
+  (symbol (lib_id "power:+3V3") (at 27.94 205.74 0) (unit 1)
+    (in_bom yes) (on_board yes)
+    (property "Reference" "#PWR?" (id 0) (at 27.94 209.55 0)
+      (effects (font (size 1.27 1.27)) hide)
+    )
+    (property "Value" "+3V3" (id 1) (at 28.321 201.3458 0))
+    (property "Footprint" "" (id 2) (at 27.94 205.74 0)
+      (effects (font (size 1.27 1.27)) hide)
+    )
+    (property "Datasheet" "" (id 3) (at 27.94 205.74 0)
+      (effects (font (size 1.27 1.27)) hide)
+    )
+    (pin "1")
+  )
   (symbol (lib_id "power:+3V3") (at 27.94 246.38 0) (unit 1)
     (in_bom yes) (on_board yes)
@@
     (pin "1")
   )
+  (symbol (lib_id "power:+3V3") (at 284.48 226.06 90) (unit 1)
+    (in_bom yes) (on_board yes)
+    (property "Reference" "#PWR?" (id 0) (at 288.29 226.06 0)
+      (effects (font (size 1.27 1.27)) hide)
+    )
+    (property "Value" "+3V3" (id 1) (at 280.0858 225.679 0))
+    (property "Footprint" "" (id 2) (at 284.48 226.06 0)
+      (effects (font (size 1.27 1.27)) hide)
+    )
+    (property "Datasheet" "" (id 3) (at 284.48 226.06 0)
+      (effects (font (size 1.27 1.27)) hide)
+    )
+    (pin "1")
+  )
   (symbol (lib_name "power:PWR_FLAG_1") (lib_id "power:PWR_FLAG") (at 137.16 46.99 0) (unit 1)
     (in_bom yes) (on_board yes)
@@
     (pin "1")
   )
-  (symbol (lib_id "power:GND") (at 27.94 207.01 0) (unit 1)
-    (in_bom yes) (on_board yes)
-    (property "Reference" "#PWR0194" (id 0) (at 27.94 213.36 0)
-      (effects (font (size 1.27 1.27)) hide)
-    )
-    (property "Value" "GND" (id 1) (at 28.067 211.4042 0))
-    (property "Footprint" "" (id 2) (at 27.94 207.01 0)
-      (effects (font (size 1.27 1.27)) hide)
-    )
-    (property "Datasheet" "" (id 3) (at 27.94 207.01 0)
-      (effects (font (size 1.27 1.27)) hide)
-    )
-    (pin "1")
-  )
   (symbol (lib_id "power:GND") (at 29.21 93.98 0) (unit 1)
     (in_bom yes) (on_board yes)
@@
   (symbol (lib_id "power:GND") (at 288.29 228.6 0) (unit 1)
     (in_bom yes) (on_board yes)
-    (property "Reference" "#PWR?" (id 0) (at 288.29 234.95 0)
+    (property "Reference" "#PWR0212" (id 0) (at 288.29 234.95 0)
       (effects (font (size 1.27 1.27)) hide)
     )
@@
   (symbol (lib_id "Connector_Generic:Conn_01x07") (at 295.91 218.44 0) (unit 1)
     (in_bom yes) (on_board yes)
-    (property "Reference" "J?" (id 0) (at 297.9166 217.3732 0)
+    (property "Reference" "J4" (id 0) (at 297.9166 217.3732 0)
       (effects (font (size 1.27 1.27)) (justify left))
     )
@@
       (reference "#PWR0193") (unit 1) (value "+3V3") (footprint "")
     )
-    (path "/3349f8a4-b793-401a-9e84-bf9fbe1234b1"
-      (reference "#PWR0194") (unit 1) (value "GND") (footprint "")
-    )
     (path "/3e45a98d-b531-4b2f-b0ca-853b321e3ca4"
       (reference "#PWR0195") (unit 1) (value "GND") (footprint "")
@@
       (reference "#PWR0211") (unit 1) (value "+1V8") (footprint "")
     )
+    (path "/31bda364-0ce6-485b-974c-c9ffebd9bcd5"
+      (reference "#PWR0212") (unit 1) (value "GND") (footprint "")
+    )
     (path "/00000000-0000-0000-0000-00005d90f565"
       (reference "#PWR0226") (unit 1) (value "GND") (footprint "")
@@
       (reference "#PWR0227") (unit 1) (value "GND") (footprint "")
     )
-    (path "/31bda364-0ce6-485b-974c-c9ffebd9bcd5"
-      (reference "#PWR?") (unit 1) (value "GND") (footprint "")
+    (path "/4cc6d7bf-e3bc-404b-a46a-09de67eef1e0"
+      (reference "#PWR?") (unit 1) (value "+3V3") (footprint "")
+    )
+    (path "/7d3e356c-3a35-4e4b-9a7b-34e9027df934"
+      (reference "#PWR?") (unit 1) (value "+3V3") (footprint "")
     )
     (path "/857280fb-7cc4-40b2-aa09-0bf266d28d37"
@@
       (reference "J3") (unit 1) (value "HDMI_A_1.4") (footprint "kimchi_ulid:HDMI-10029449-111RLF")
     )
+    (path "/25679d49-e193-4417-8b08-52a6d54eea1f"
+      (reference "J4") (unit 1) (value "Jtag") (footprint "Connector_PinHeader_2.54mm:PinHeader_1x07_P2.54mm_Vertical")
+    )
     (path "/049ca297-7319-4484-90e0-aca9d4f8f519"
       (reference "J5") (unit 1) (value "Flash") (footprint "Connector_PinHeader_2.54mm:PinHeader_1x07_P2.54mm_Vertical")
     )
-    (path "/25679d49-e193-4417-8b08-52a6d54eea1f"
-      (reference "J?") (unit 1) (value "Jtag") (footprint "Connector_PinHeader_2.54mm:PinHeader_1x07_P2.54mm_Vertical")
-    )
     (path "/00000000-0000-0000-0000-000060d1af4a"
